Commit message: Added IMU sensor

File: racecar_gazebo/racecar_description/urdf/racecar.xacro (robot description, xacro)
@@ -5,4 +5,5 @@
   <xacro:arg name="color" default="blue" />
   <xacro:property name="color" value="$(arg color)" />
+  <xacro:property name="dummy_inertia" value="1e-09"/>
   <xacro:include filename="$(find racecar_description)/urdf/macros.xacro" />
   <!-- Add chassis and it's inertia link -->
@@ -29,4 +30,15 @@
     </inertial>
   </link>
+  <link name="${robot_name}/imu_link">
+    <inertial>
+      <mass value="0.001"/>
+      <origin xyz="0 0 0" rpy="0 0 0"/>
+      <inertia ixx="${dummy_inertia}" ixy="0.0" ixz="0.0" iyy="${dummy_inertia}" iyz="0.0" izz="${dummy_inertia}"/>
+    </inertial>
+  </link>
+  <joint name="${robot_name}/imu_joint" type="fixed">
+    <parent link="${robot_name}/chassis" />
+    <child link="${robot_name}/imu_link" />
+  </joint>
   <joint name="${robot_name}/chassis_inertia_joint" type="fixed">
     <origin xyz="0 0 0" rpy="0 0 0" />

Commit message: Code cleanup

File: racecar_gazebo/racecar_description/urdf/racecar.xacro (robot description, xacro)
@@ -191,8 +191,10 @@
     <axis xyz="0 0 1" />
   </joint>
-  <xacro:include filename="$(find racecar_description)/urdf/include/_d435.urdf.xacro" />
-  <xacro:sensor_d435 parent="${robot_name}/chassis" name="${robot_name}/camera" topics_ns="$(arg robot_name)">
-    <origin xyz="0.390 0 0.04" rpy="0 0 0"/>
-  </xacro:sensor_d435>
+  <xacro:unless value="$(optenv DISABLE_GAZEBO_CAMERA false)">
+    <xacro:include filename="$(find racecar_description)/urdf/include/_d435.urdf.xacro" />
+    <xacro:sensor_d435 parent="${robot_name}/chassis" name="${robot_name}/camera" topics_ns="$(arg robot_name)">
+      <origin xyz="0.390 0 0.04" rpy="0 0 0"/>
+    </xacro:sensor_d435>
+  </xacro:unless>
   <!-- zed camera -->
 <!--  <link name="zed_camera_link">-->

Commit message: Update racecar.xacro

File: racecar_gazebo/racecar_description/urdf/racecar.xacro (robot description, xacro)
@@ -9,14 +9,4 @@
   <!-- Add chassis and it's inertia link -->
   <link name="${robot_name}/base_link" />
-  <!-- If blue, include urdf/include/chassis_blue.xacro, else if red, include urdf/include/chassis_red.xacro -->
-<!--  <xacro:if value="${color == 'blue'}">-->
-<!--    <xacro:include filename="$(find racecar_description)/urdf/include/chassis_blue.xacro" />-->
-<!--  </xacro:if>-->
-<!--  <xacro:if value="${color == 'red'}">-->
-<!--    <xacro:include filename="$(find racecar_description)/urdf/include/chassis_red.xacro" />-->
-<!--  </xacro:if>-->
-<!--  <xacro:if value="${color == 'green'}">-->
-<!--    <xacro:include filename="$(find racecar_description)/urdf/include/chassis_green.xacro" />-->
-<!--  </xacro:if>-->
   <xacro:chassis color="${color}" robot_name="${robot_name}" />
   <joint name="${robot_name}/base_link_joint" type="fixed">
@@ -116,5 +106,5 @@
     </visual>
   </link>
-  <joint name="${robot_name}/right_steering_hinge_joint" type="continuous">
+  <joint name="${robot_name}/right_steering_hinge_joint" type="revolute">
     <origin xyz="0.325 -0.1 0" rpy="0 1.5708 0" />
     <parent link="${robot_name}/chassis" />
@@ -197,60 +187,4 @@
     </xacro:sensor_d435>
   </xacro:unless>
-  <!-- zed camera -->
-<!--  <link name="zed_camera_link">-->
-<!--    <inertial>-->
-<!--      <mass value="1e-5" />-->
-<!--      <origin xyz="0 0 0" rpy="0 0 0"/>-->
-<!--      <inertia ixx="1e-6" ixy="0" ixz="0" iyy="1e-6" iyz="0" izz="1e-6" />-->
-<!--    </inertial>-->
-<!--    <collision>-->
-<!--      <origin xyz="0 0 0" rpy="0 0 0"/>-->
-<!--      <geometry>-->
-<!--        <box size="0.033 0.175 0.030"/>-->
-<!--      </geometry>-->
-<!--    </collision>-->
-<!--    <visual>-->
-<!--      <origin xyz="0 0 0" rpy="0 0 0"/>-->
-<!--      <geometry>-->
-<!--        <box size="0.033 0.175 0.030"/>-->
-<!--      </geometry>-->
-<!--      <material name="red"/>-->
-<!--    </visual>-->
-<!--  </link>-->
-<!--  <joint name="zed_camera_joint" type="fixed">-->
-<!--    <origin xyz="0.390 0 0.04" rpy="0 0 0"/>-->
-<!--    <parent link="chassis"/>-->
-<!--    <child link="zed_camera_link"/>-->
-<!--    <axis xyz="0 0 1" />-->
-<!--    &lt;!&ndash; <limit lower="0.0" upper="0.0" effort="0.0" velocity="0.0" /> &ndash;&gt;-->
-<!--  </joint>-->
-<!--  &lt;!&ndash; zed camera lenses &ndash;&gt;-->
-<!--  &lt;!&ndash; It seems these have to have a non-zero mass to have a camera attached? &ndash;&gt;-->
-<!--  <link name="camera_link">&lt;!&ndash; this needs to match the name in zed_wrapper/zed_tf.launch &ndash;&gt;-->
-<!--    <inertial>-->
-<!--      <mass value="1e-5" />-->
-<!--      <origin xyz="0 0 0" rpy="0 0 0"/>-->
-<!--      <inertia ixx="1e-6" ixy="0" ixz="0" iyy="1e-6" iyz="0" izz="1e-6" />-->
-<!--    </inertial>-->
-<!--  </link>-->
-<!--  <link name="zed_camera_right_link">-->
-<!--    <inertial>-->
-<!--      <mass value="1e-5" />-->
-<!--      <origin xyz="0 0 0" rpy="0 0 0"/>-->
-<!--      <inertia ixx="1e-6" ixy="0" ixz="0" iyy="1e-6" iyz="0" izz="1e-6" />-->
-<!--    </inertial>-->
-<!--  </link>-->
-<!--  <joint name="zed_camera_left_joint" type="fixed">-->
-<!--    <origin xyz="0 0.06 0" rpy="0 0 0"/>-->
-<!--    <parent link="zed_camera_link"/>-->
-<!--    <child link="camera_link"/>-->
-<!--    <axis xyz="0 0 1" />-->
-<!--  </joint>-->
-<!--  <joint name="zed_camera_right_joint" type="fixed">-->
-<!--    <origin xyz="0 -0.06 0" rpy="0 0 0"/>-->
-<!--    <parent link="zed_camera_link"/>-->
-<!--    <child link="zed_camera_right_link"/>-->
-<!--    <axis xyz="0 0 1" />-->
-<!--  </joint>-->
   <!-- Add the remaining xacros -->
   <xacro:include filename="$(find racecar_description)/urdf/racecar.gazebo" />
